File: pcb/watch.kicad_sch (KiCad schematic)
At the start: 14 parts, among them SW1 SW_Push, U1 ATtiny84A-P, U3 LTC-4627JD, Y1 Crystal

Commit message: Update schematic diagram + readme
Parts:
- U3: value LTC-4627JD -> ~
- Y1: value Crystal -> 32KHz
Other:
- moved on the sheet: Y1
Changed lines of the file:
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@@
 	(wire
 		(pts
-			(xy 76.2 71.12) (xy 82.55 71.12)
+			(xy 76.2 72.39) (xy 82.55 72.39)
 		)
 		(stroke
@@
 	(wire
 		(pts
-			(xy 82.55 78.74) (xy 82.55 80.01)
-		)
-		(stroke
-			(width 0)
-			(type default)
-		)
-	)
-	(wire
-		(pts
 			(xy 102.87 50.8) (xy 128.27 50.8)
 		)
@@
 	(wire
 		(pts
-			(xy 76.2 71.12) (xy 76.2 74.93)
+			(xy 76.2 72.39) (xy 76.2 74.93)
 		)
 		(stroke
@@
 		(fields_autoplaced yes)
 		(property "Reference" "U3"
-			(at 151.13 50.8 0)
-			(effects
-				(font
-					(size 1.27 1.27)
-				)
-			)
-		)
-		(property "Value" "LTC-4627JD"
 			(at 151.13 53.34 0)
 			(effects
@@
 					(size 1.27 1.27)
 				)
+			)
+		)
+		(property "Value" "~"
+			(at 151.13 53.34 0)
+			(effects
+				(font
+					(size 1.27 1.27)
+				)
+				(hide yes)
 			)
 		)
@@
 	(symbol
 		(lib_id "Device:Crystal")
-		(at 82.55 74.93 90)
+		(at 82.55 76.2 90)
 		(unit 1)
 		(exclude_from_sim no)
@@
 		(fields_autoplaced yes)
 		(property "Reference" "Y1"
-			(at 86.36 73.6599 90)
+			(at 86.36 74.9299 90)
 			(effects
 				(font
@@
 			)
 		)
-		(property "Value" "Crystal"
-			(at 86.36 76.1999 90)
+		(property "Value" "32KHz"
+			(at 86.36 77.4699 90)
 			(effects
 				(font
@@
 		)
 		(property "Footprint" "Crystal:Crystal_Round_D1.5mm_Vertical"
-			(at 82.55 74.93 0)
+			(at 82.55 76.2 0)
 			(effects
 				(font
@@
 		)
 		(property "Datasheet" "~"
-			(at 82.55 74.93 0)
+			(at 82.55 76.2 0)
 			(effects
 				(font
@@
 		)
 		(property "Description" "Two pin crystal"
-			(at 82.55 74.93 0)
-			(effects
-				(font
+			(at 82.55 76.2 0)
+			(effects
+				(font
